File: Flex debug cable/Flex debug cable.kicad_sch (KiCad schematic)
At the start: 4 parts, among them J2 FPC 10P, J3 B2B GT-B0353FSV06-06B0201, J4 B2B GT-B0353FSV06-08B0201, J5 B2B YXT-BB10-10S-02

Commit message: Design flex debug cable V1.1
Parts:
- removed J3: B2B GT-B0353FSV06-06B0201, Picoballoon Mechanical & Misc:B2B GT-B0353FSV06-06B0201, symbol Picoballoon Mechanical & Misc:B2B GT-B0353FSV06-06B0201
- removed J5: B2B YXT-BB10-10S-02, Picoballoon Mechanical & Misc:B2B YXT-BB10-10S-02, symbol Picoballoon Mechanical & Misc:B2B YXT-BB10-10S-02
Other:
- note removed: "10P 0.4mm B2B connector"
- note removed: "8P 0.35mm B2B connector"
- moved on the sheet: J2, J4
