File: Flex debug cable/Flex debug cable.kicad_pcb (KiCad board)
At the start: 2 copper layers, 100 x 5.5 mm, 5 parts, among them J2 FPC 10P, J3 B2B GT-B0353FSV06-06B0201, J4 B2B GT-B0353FSV06-08B0201, J5 B2B YXT-BB10-10S-02

Commit message: Design flex debug cable V1.1
Parts:
- removed J3: B2B GT-B0353FSV06-06B0201, Picoballoon Mechanical & Misc:B2B GT-B0353FSV06-06B0201
- removed J5: B2B YXT-BB10-10S-02, Picoballoon Mechanical & Misc:B2B YXT-BB10-10S-02
- moved J4 4.55 mm to (148.4, 75.0)
Routing:
- net GND: track 87.2 -> 95.3 mm
- net /SWDIO: track 102.7 -> 97.0 mm, vias 3 -> 1
- net /RST: track 102.5 -> 97.4 mm, vias 2 -> 1
- net /SWDCLK: track 100.4 -> 97.1 mm, vias 3 -> 1
- net /SWO: track 99.3 -> 97.3 mm, vias 2 -> 1
- net V_SOLAR: track 100.8 -> 99.1 mm, vias 3 -> 1
- net /TG_RX: track 97.6 -> 99.0 mm, vias 2 -> 1
- net V_TARGET: track 100.7 -> 99.3 mm, vias 3 -> 1
- net /TG_TX: track 98.8 -> 98.7 mm, vias 2 -> 1
Other:
- board text added: "Flex debug cable V1.1"
- board text removed: "Flex debug cable V1.0"
