File: Integrated Debugger/MCU.kicad_sch (KiCad schematic)
At the start: 14 parts, among them SW1 BOOT, U2 STM32F103CBUx, Y1 8MHz

Commit message: Update BOM
Parts:
- C1, C2, C3, C4, C5: LCSC Part # C76934 -> C181043; MPN GRM033R61A104KE15D -> GRM033R6YA104KE14D
- C6: LCSC Part # C76930 -> C335102; MPN GRM033R60J105MEA2D -> GRM033R61C105ME15D
- renumbered R9 to R10, R10 to R11, R11 to R12, R8 to R9
Changed lines of the file:
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@@
 			)
 		)
-		(property "Datasheet" "~"
+		(property "Datasheet" "https://jlcpcb.com/api/file/downloadByFileSystemAccessId/8588903659258458112"
 			(at 171.45 67.31 0)
 			(effects
@@
 			)
 		)
-		(property "MPN" "GRM033R61A104KE15D"
+		(property "MPN" "GRM033R6YA104KE14D"
 			(at 171.45 67.31 0)
 			(effects
@@
 			)
 		)
-		(property "LCSC Part #" "C76934"
+		(property "LCSC Part #" "C181043"
 			(at 171.45 67.31 90)
 			(effects
@@
 			)
 		)
-		(property "Datasheet" "~"
+		(property "Datasheet" "https://jlcpcb.com/api/file/downloadByFileSystemAccessId/8588903659258458112"
 			(at 107.95 27.94 0)
 			(effects
@@
 			)
 		)
-		(property "MPN" "GRM033R61A104KE15D"
+		(property "MPN" "GRM033R6YA104KE14D"
 			(at 107.95 27.94 0)
 			(effects
@@
 			)
 		)
-		(property "LCSC Part #" "C76934"
+		(property "LCSC Part #" "C181043"
 			(at 107.95 27.94 0)
 			(effects
@@
 			)
 		)
-		(property "Datasheet" "~"
+		(property "Datasheet" "https://jlcpcb.com/api/file/downloadByFileSystemAccessId/8588903659258458112"
 			(at 171.45 36.83 0)
 			(effects
@@
 			)
 		)
-		(property "MPN" "GRM033R61A104KE15D"
+		(property "MPN" "GRM033R6YA104KE14D"
 			(at 171.45 36.83 0)
 			(effects
@@
 			)
 		)
-		(property "LCSC Part #" "C76934"
+		(property "LCSC Part #" "C181043"
 			(at 171.45 36.83 90)
 			(effects
@@
 			)
 		)
-		(property "Datasheet" "~"
+		(property "Datasheet" "https://jlcpcb.com/api/file/downloadByFileSystemAccessId/8588954991717453824"
 			(at 171.45 77.47 0)
 			(effects
@@
 			)
 		)
-		(property "MPN" "GRM033R60J105MEA2D"
+		(property "MPN" "GRM033R61C105ME15D"
 			(at 171.45 77.47 0)
 			(effects
@@
 			)
 		)
-		(property "LCSC Part #" "C76930"
+		(property "LCSC Part #" "C335102"
 			(at 171.45 77.47 90)
 			(effects
@@
 		(dnp no)
 		(fields_autoplaced yes)
-		(property "Reference" "R10"
+		(property "Reference" "R11"
 			(at 116.84 49.8475 0)
 			(do_not_autoplace yes)
@@
 			(project "Integrated Debugger"
 				(path "/ce538ebe-fda9-4af3-9f8c-9fd5bf58f0e4/b916d44a-03d1-4a04-a023-19b38caca2ea"
-					(reference "R10")
+					(reference "R11")
 					(unit 1)
 				)
@@
 			)
 		)
-		(property "Datasheet" "~"
+		(property "Datasheet" "https://jlcpcb.com/api/file/downloadByFileSystemAccessId/8588903659258458112"
 			(at 171.45 46.99 0)
 			(effects
@@
 			)
 		)
-		(property "MPN" "GRM033R61A104KE15D"
+		(property "MPN" "GRM033R6YA104KE14D"
 			(at 171.45 46.99 0)
 			(effects
@@
 			)
 		)
-		(property "LCSC Part #" "C76934"
+		(property "LCSC Part #" "C181043"
 			(at 171.45 46.99 90)
 			(effects
@@
 			)
 		)
-		(property "Datasheet" "~"
+		(property "Datasheet" "https://jlcpcb.com/api/file/downloadByFileSystemAccessId/8588903659258458112"
 			(at 171.45 57.15 0)
 			(effects
@@
 			)
 		)
-		(property "MPN" "GRM033R61A104KE15D"
+		(property "MPN" "GRM033R6YA104KE14D"
 			(at 171.45 57.15 0)
 			(effects
@@
 			)
 		)
-		(property "LCSC Part #" "C76934"
+		(property "LCSC Part #" "C181043"
 			(at 171.45 57.15 90)
 			(effects
@@
 		(on_board yes)
 		(dnp no)
-		(property "Reference" "R8"
+		(property "Reference" "R9"
 			(at 84.074 75.184 90)
 			(do_not_autoplace yes)
@@
 			(project "Integrated Debugger"
 				(path "/ce538ebe-fda9-4af3-9f8c-9fd5bf58f0e4/b916d44a-03d1-4a04-a023-19b38caca2ea"
-					(reference "R8")
+					(reference "R9")
 					(unit 1)
 				)
@@
 		(dnp no)
 		(fields_autoplaced yes)
-		(property "Reference" "R11"
+		(property "Reference" "R12"
 			(at 116.84 65.0875 0)
 			(do_not_autoplace yes)
@@
 			(project "Integrated Debugger"
 				(path "/ce538ebe-fda9-4af3-9f8c-9fd5bf58f0e4/b916d44a-03d1-4a04-a023-19b38caca2ea"
-					(reference "R11")
+					(reference "R12")
 					(unit 1)
 				)
@@
 			)
 		)
-		(property "Datasheet" "~"
+		(property "Datasheet" "https://jlcpcb.com/api/file/downloadByFileSystemAccessId/8589041619525492736"
 			(at 171.45 87.63 0)
 			(effects
@@
 		(dnp no)
 		(fields_autoplaced yes)
-		(property "Reference" "R9"
+		(property "Reference" "R10"
 			(at 95.25 80.3275 0)
 			(do_not_autoplace yes)
@@
 			(project "Integrated Debugger"
 				(path "/ce538ebe-fda9-4af3-9f8c-9fd5bf58f0e4/b916d44a-03d1-4a04-a023-19b38caca2ea"
-					(reference "R9")
-					(unit 1)
-				)
+					(reference "R10")
+					(unit 1)
+				)

Commit message: feat: fix debugger bugs & impl. auxiliary power - 869b0p9f3
Parts:
- added C17: 100nF, Picoballoon Passives:Capacitor 0201, symbol Picoballoon Passives:Capacitor
- R9: now not fitted
Connections:
- net GND: now also C17.1
- net VBUS: no longer R11.1
- net at R11.2, R12.1, U2.18 (PB0): now also C17.2
- net SOL_EN renamed AUX_EN
- new net V_TARGET: R11.1
Other:
- moved on the sheet: R11, R12
