File: Integrated Debugger/MCU.kicad_sch (KiCad schematic)
At the start: 17 parts, among them SW1 BOOT, U2 STM32F103CBUx, Y1 8MHz

Commit message: capacitors updated
Parts:
- C10, C12: value 18pF -> 15pF; LCSC Part # C161409 -> C1853525; MPN GRM0335C1H180GA01D -> CC0201GRNPO8BN150
Changed lines of the file:
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@@
 			)
 		)
-		(property "Value" "18pF"
+		(property "Value" "15pF"
 			(at 109.855 123.825 0)
 			(effects
@@
 			)
 		)
-		(property "MPN" "GRM0335C1H180GA01D"
+		(property "MPN" "CC0201GRNPO8BN150"
 			(at 109.22 121.92 0)
 			(effects
@@
 			)
 		)
-		(property "LCSC Part #" "C161409"
+		(property "LCSC Part #" "C1853525"
 			(at 109.22 121.92 0)
 			(effects
@@
 			)
 		)
-		(property "Value" "18pF"
+		(property "Value" "15pF"
 			(at 98.425 123.825 0)
 			(effects
@@
 			)
 		)
-		(property "MPN" "GRM0335C1H180GA01D"
+		(property "MPN" "CC0201GRNPO8BN150"
 			(at 99.06 121.92 0)
 			(effects
@@
 			)
 		)
-		(property "LCSC Part #" "C161409"
+		(property "LCSC Part #" "C1853525"
 			(at 99.06 121.92 0)
 			(effects
