File: Integrated Debugger/Integrated Debugger.kicad_sch (KiCad schematic)
At the start: 20 parts, among them J1 B2B GT-B0353FSV06-08B0201, J6 TYPE-C-31-M-12, U5 USBLC6-2P6

Commit message: Reannotate schematic, update GND plane
Parts:
- renumbered C9 to C1, C8 to C2, D2 to D1, D3 to D2, D4 to D3, J6 to J2, R15 to R10, R14 to R11, R20 to R4, R21 to R5, R5 to R6, R6 to R7, R4 to R8, R22 to R9, U5 to U1
Changed lines of the file:
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@@
 		(on_board yes)
 		(dnp no)
-		(property "Reference" "J6"
+		(property "Reference" "J2"
 			(at 226.06 101.6 0)
 			(effects
@@
 			(project "Integrated Debugger"
 				(path "/ce538ebe-fda9-4af3-9f8c-9fd5bf58f0e4"
-					(reference "J6")
+					(reference "J2")
 					(unit 1)
 				)
@@
 		(dnp no)
 		(fields_autoplaced yes)
-		(property "Reference" "R21"
+		(property "Reference" "R5"
 			(at 163.83 72.7075 0)
 			(do_not_autoplace yes)
@@
 			(project "Integrated Debugger"
 				(path "/ce538ebe-fda9-4af3-9f8c-9fd5bf58f0e4"
-					(reference "R21")
+					(reference "R5")
 					(unit 1)
 				)
@@
 		(dnp no)
 		(fields_autoplaced yes)
-		(property "Reference" "#PWR04"
+		(property "Reference" "#PWR03"
 			(at 105.41 134.62 0)
 			(effects
@@
 			(project "Programmer"
 				(path "/ce538ebe-fda9-4af3-9f8c-9fd5bf58f0e4"
-					(reference "#PWR04")
+					(reference "#PWR03")
 					(unit 1)
 				)
@@
 		(on_board yes)
 		(dnp no)
-		(property "Reference" "D4"
+		(property "Reference" "D3"
 			(at 72.39 80.01 0)
 			(do_not_autoplace yes)
@@
 			(project "Programmer"
 				(path "/ce538ebe-fda9-4af3-9f8c-9fd5bf58f0e4"
-					(reference "D4")
+					(reference "D3")
 					(unit 1)
 				)
@@
 		(on_board yes)
 		(dnp no)
-		(property "Reference" "#PWR053"
+		(property "Reference" "#PWR07"
 			(at 186.69 151.13 0)
 			(effects
@@
 			(project "Integrated Debugger"
 				(path "/ce538ebe-fda9-4af3-9f8c-9fd5bf58f0e4"
-					(reference "#PWR053")
+					(reference "#PWR07")
 					(unit 1)
 				)
@@
 		(on_board yes)
 		(dnp no)
-		(property "Reference" "R15"
+		(property "Reference" "R10"
 			(at 193.04 137.4775 0)
 			(do_not_autoplace yes)
@@
 			(project "Integrated Debugger"
 				(path "/ce538ebe-fda9-4af3-9f8c-9fd5bf58f0e4"
-					(reference "R15")
+					(reference "R10")
 					(unit 1)
 				)
@@
 		(on_board yes)
 		(dnp no)
-		(property "Reference" "R6"
+		(property "Reference" "R7"
 			(at 170.18 120.396 90)
 			(do_not_autoplace yes)
@@
 			(project "Programmer"
 				(path "/ce538ebe-fda9-4af3-9f8c-9fd5bf58f0e4"
-					(reference "R6")
+					(reference "R7")
 					(unit 1)
 				)
@@
 		(on_board yes)
 		(dnp no)
-		(property "Reference" "#PWR03"
+		(property "Reference" "#PWR02"
 			(at 93.98 125.73 0)
 			(effects
@@
 			(project "Programmer"
 				(path "/ce538ebe-fda9-4af3-9f8c-9fd5bf58f0e4"
-					(reference "#PWR03")
+					(reference "#PWR02")
 					(unit 1)
 				)
@@
 		(on_board yes)
 		(dnp no)
-		(property "Reference" "R5"
+		(property "Reference" "R6"
 			(at 170.18 111.506 90)
 			(do_not_autoplace yes)
@@
 			(project "Programmer"
 				(path "/ce538ebe-fda9-4af3-9f8c-9fd5bf58f0e4"
-					(reference "R5")
+					(reference "R6")
 					(unit 1)
 				)
@@
 		(on_board yes)
 		(dnp no)
-		(property "Reference" "C9"
+		(property "Reference" "C1"
 			(at 187.96 102.87 90)
 			(do_not_autoplace yes)
@@
 			(project "Integrated Debugger"
 				(path "/ce538ebe-fda9-4af3-9f8c-9fd5bf58f0e4"
-					(reference "C9")
+					(reference "C1")
 					(unit 1)
 				)
@@
 		(dnp no)
 		(fields_autoplaced yes)
-		(property "Reference" "R20"
+		(property "Reference" "R4"
 			(at 163.83 65.0875 0)
 			(do_not_autoplace yes)
@@
 			(project "Integrated Debugger"
 				(path "/ce538ebe-fda9-4af3-9f8c-9fd5bf58f0e4"
-					(reference "R20")
+					(reference "R4")
 					(unit 1)
 				)
@@
 		(on_board yes)
 		(dnp no)
-		(property "Reference" "#PWR056"
+		(property "Reference" "#PWR06"
 			(at 176.53 107.95 0)
 			(effects
@@
 			(project "Integrated Debugger"
 				(path "/ce538ebe-fda9-4af3-9f8c-9fd5bf58f0e4"
-					(reference "#PWR056")
+					(reference "#PWR06")
 					(unit 1)
 				)
@@
 		(on_board yes)
 		(dnp no)
-		(property "Reference" "D2"
+		(property "Reference" "D1"
 			(at 72.39 64.77 0)
 			(do_not_autoplace yes)
@@
 			(project "Programmer"
 				(path "/ce538ebe-fda9-4af3-9f8c-9fd5bf58f0e4"
-					(reference "D2")
+					(reference "D1")
 					(unit 1)
 				)
@@
 		(on_board yes)
 		(dnp no)
-		(property "Reference" "U5"
+		(property "Reference" "U1"
 			(at 194.31 111.125 0)
 			(effects
@@
 			(project "Integrated Debugger"
 				(path "/ce538ebe-fda9-4af3-9f8c-9fd5bf58f0e4"
-					(reference "U5")
+					(reference "U1")
 					(unit 1)
 				)
@@
 		(dnp no)
 		(fields_autoplaced yes)
-		(property "Reference" "#PWR02"
+		(property "Reference" "#PWR01"
 			(at 64.77 92.71 0)
 			(effects
@@
 			(project ""
 				(path "/ce538ebe-fda9-4af3-9f8c-9fd5bf58f0e4"
-					(reference "#PWR02")
+					(reference "#PWR01")
 					(unit 1)
 				)
@@
 		(on_board yes)
 		(dnp no)
-		(property "Reference" "#PWR020"
+		(property "Reference" "#PWR013"
 			(at 223.52 166.37 0)
 			(effects
@@
 			(project "Integrated Debugger"
 				(path "/ce538ebe-fda9-4af3-9f8c-9fd5bf58f0e4"
-					(reference "#PWR020")
+					(reference "#PWR013")
 					(unit 1)
 				)
@@
 		(on_board yes)
 		(dnp no)
-		(property "Reference" "#PWR032"
+		(property "Reference" "#PWR012"
 			(at 218.44 166.37 0)
 			(effects
@@
 			(project "Integrated Debugger"
 				(path "/ce538ebe-fda9-4af3-9f8c-9fd5bf58f0e4"
-					(reference "#PWR032")
+					(reference "#PWR012")
 					(unit 1)
 				)
@@
 		(on_board yes)
 		(dnp no)
-		(property "Reference" "#PWR033"
+		(property "Reference" "#PWR011"
 			(at 215.9 149.86 0)
 			(effects
@@
 			(project "Integrated Debugger"
 				(path "/ce538ebe-fda9-4af3-9f8c-9fd5bf58f0e4"
-					(reference "#PWR033")
+					(reference "#PWR011")
 					(unit 1)
 				)
@@
 		(on_board yes)
 		(dnp no)
-		(property "Reference" "D3"
+		(property "Reference" "D2"
 			(at 72.39 72.39 0)
 			(do_not_autoplace yes)
@@
 			(project "Programmer"
 				(path "/ce538ebe-fda9-4af3-9f8c-9fd5bf58f0e4"
-					(reference "D3")
+					(reference "D2")
 					(unit 1)
 				)
@@
 		(dnp no)
 		(fields_autoplaced yes)
-		(property "Reference" "#PWR050"
+		(property "Reference" "#PWR05"
 			(at 162.56 83.82 0)
 			(effects
@@
 			(project "Integrated Debugger"
 				(path "/ce538ebe-fda9-4af3-9f8c-9fd5bf58f0e4"
-					(reference "#PWR050")
+					(reference "#PWR05")
 					(unit 1)
 				)
@@
 		(on_board yes)
 		(dnp no)
-		(property "Reference" "R4"
+		(property "Reference" "R8"
 			(at 170.18 128.27 90)
 			(do_not_autoplace yes)
@@
 			(project "Integrated Debugger"
 				(path "/ce538ebe-fda9-4af3-9f8c-9fd5bf58f0e4"
-					(reference "R4")
+					(reference "R8")
 					(unit 1)
 				)
@@
 		(dnp no)
 		(fields_autoplaced yes)
-		(property "Reference" "C8"
+		(property "Reference" "C2"
 			(at 217.805 153.035 0)
 			(do_not_autoplace yes)
@@
 			(project "Integrated Debugger"
 				(path "/ce538ebe-fda9-4af3-9f8c-9fd5bf58f0e4"
-					(reference "C8")
+					(reference "C2")
 					(unit 1)
 				)
@@
 		(dnp no)
 		(fields_autoplaced yes)
-		(property "Reference" "R22"
+		(property "Reference" "R9"
 			(at 185.42 137.4775 0)
 			(do_not_autoplace yes)
@@
 			(project "Integrated Debugger"
 				(path "/ce538ebe-fda9-4af3-9f8c-9fd5bf58f0e4"
-					(reference "R22")
+					(reference "R9")
 					(unit 1)
 				)
@@
 		(on_board yes)
 		(dnp no)
-		(property "Reference" "#PWR049"
+		(property "Reference" "#PWR04"
 			(at 162.56 66.04 0)
 			(effects
@@
 			(project "Integrated Debugger"
 				(path "/ce538ebe-fda9-4af3-9f8c-9fd5bf58f0e4"
-					(reference "#PWR049")
+					(reference "#PWR04")
 					(unit 1)
 				)
@@
 		(on_board yes)
 		(dnp no)
-		(property "Reference" "#PWR051"
+		(property "Reference" "#PWR010"
 			(at 193.04 129.54 0)
 			(effects
@@
 			(project "Integrated Debugger"
 				(path "/ce538ebe-fda9-4af3-9f8c-9fd5bf58f0e4"
-					(reference "#PWR051")
+					(reference "#PWR010")
 					(unit 1)
 				)
@@
 		(on_board yes)
 		(dnp no)
-		(property "Reference" "R14"
+		(property "Reference" "R11"
 			(at 224.79 153.9875 0)
 			(do_not_autoplace yes)
@@
 			(project "Integrated Debugger"
 				(path "/ce538ebe-fda9-4af3-9f8c-9fd5bf58f0e4"
-					(reference "R14")
+					(reference "R11")
 					(unit 1)
 				)
@@
 		(on_board yes)
 		(dnp no)
-		(property "Reference" "#PWR052"
+		(property "Reference" "#PWR08"
 			(at 191.77 151.13 0)
 			(effects
@@
 			(project "Integrated Debugger"
 				(path "/ce538ebe-fda9-4af3-9f8c-9fd5bf58f0e4"
-					(reference "#PWR052")
+					(reference "#PWR08")
 					(unit 1)
 				)
@@
 		(on_board yes)
 		(dnp no)
-		(property "Reference" "#PWR054"
+		(property "Reference" "#PWR09"
 			(at 193.04 102.87 0)
 			(effects
@@
 			(project "Integrated Debugger"
 				(path "/ce538ebe-fda9-4af3-9f8c-9fd5bf58f0e4"
-					(reference "#PWR054")
-					(unit 1)
-				)
+					(reference "#PWR09")
+					(unit 1)
+				)

Commit message: led+ resistors updated
Parts:
- D1: LCSC Part # C3646923 -> C2852592; MPN XL-0201SURC -> APHHS1005SURCK
- D2: LCSC Part # C5366341 -> C5875752; MPN APG0603ZGC-5MAV -> APHHS1005LZGCK-V
- D3: LCSC Part # C3646921 -> C5354973; MPN XL-0201UBC -> APHHS1005LQBC/D-V
- R1: value 560Ω -> 1kΩ; MPN RC0201FR-07560RL -> RC0201FR-071KL
- R2: value 470Ω -> 4.7kΩ; LCSC Part # C852285 -> C138135; MPN RT0201DRD07470RL -> RC0201FR-074K7L
- R3: value 470Ω -> 220Ω; LCSC Part # C852285 -> C226657; MPN RT0201DRD07470RL -> AC0201JR-07220RL
Changed lines of the file:
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@@
 			)
 		)
-		(property "LCSC Part #" "C3646921"
+		(property "LCSC Part #" "C5354973"
 			(at 72.39 82.55 0)
 			(effects
@@
 			)
 		)
-		(property "MPN" "XL-0201UBC"
+		(property "MPN" "APHHS1005LQBC/D-V"
 			(at 72.39 82.55 0)
 			(effects
@@
 			)
 		)
-		(property "Value" "560Ω"
+		(property "Value" "1kΩ"
 			(at 83.82 64.77 90)
 			(do_not_autoplace yes)
@@
 			)
 		)
-		(property "MPN" "RC0201FR-07560RL"
+		(property "MPN" "RC0201FR-071KL"
 			(at 83.82 67.31 0)
 			(effects
@@
 			)
 		)
-		(property "LCSC Part #" "C3646923"
+		(property "LCSC Part #" "C2852592"
 			(at 72.39 67.31 0)
 			(effects
@@
 			)
 		)
-		(property "MPN" "XL-0201SURC"
+		(property "MPN" "APHHS1005SURCK"
 			(at 72.39 67.31 0)
 			(effects
@@
 			)
 		)
-		(property "Value" "470Ω"
+		(property "Value" "220Ω"
 			(at 83.82 80.01 90)
 			(do_not_autoplace yes)
@@
 			)
 		)
-		(property "MPN" "RT0201DRD07470RL"
+		(property "MPN" "AC0201JR-07220RL"
 			(at 83.82 82.55 0)
 			(effects
@@
 			)
 		)
-		(property "LCSC Part #" "C852285"
+		(property "LCSC Part #" "C226657"
 			(at 83.82 82.55 90)
 			(effects
@@
 			)
 		)
-		(property "Value" "470Ω"
+		(property "Value" "4.7kΩ"
 			(at 83.947 72.39 90)
 			(do_not_autoplace yes)
@@
 			)
 		)
-		(property "MPN" "RT0201DRD07470RL"
+		(property "MPN" "RC0201FR-074K7L"
 			(at 83.82 74.93 0)
 			(effects
@@
 			)
 		)
-		(property "LCSC Part #" "C852285"
+		(property "LCSC Part #" "C138135"
 			(at 83.82 74.93 90)
 			(effects
@@
 			)
 		)
-		(property "LCSC Part #" "C5366341"
+		(property "LCSC Part #" "C5875752"
 			(at 72.39 74.93 0)
 			(effects
@@
 			)
 		)
-		(property "MPN" "APG0603ZGC-5MAV"
+		(property "MPN" "APHHS1005LZGCK-V"
 			(at 72.39 74.93 0)
 			(effects

Commit message: IDBG v2.0 production files
Parts:
- R1: LCSC Part # C295808 -> C138165
- U1: footprint Picoballoon ICs:SOT-666-6 -> Picoballoon ICs:XSON-6; LCSC Part # C15999 -> C2999115; MPN USBLC6-2P6 -> USBULC6-2M6
Changed lines of the file:
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@@
 			)
 		)
-		(property "LCSC Part #" "C295808"
+		(property "LCSC Part #" "C138165"
 			(at 83.82 67.31 90)
 			(effects
@@
 			)
 		)
-		(property "Footprint" "Picoballoon ICs:SOT-666-6"
+		(property "Footprint" "Picoballoon ICs:XSON-6"
 			(at 191.77 121.92 0)
 			(effects
@@
 			)
 		)
-		(property "LCSC Part #" "C15999"
+		(property "LCSC Part #" "C2999115"
 			(at 193.04 115.57 0)
 			(effects
@@
 			)
 		)
-		(property "MPN" "USBLC6-2P6"
+		(property "MPN" "USBULC6-2M6"
 			(at 193.04 115.57 0)
 			(effects
