File: Integrated Debugger/Power.kicad_sch (KiCad schematic)
At the start: 25 parts, among them J5 PWR, SW3 AUXILIARY POWER, SW4 Target Override, U4 TPS22916, U5 MAX40200, U6 TPS7A2633DRVR, U7 TPS22916

Commit message: IDBG v2.0 production files
Parts:
- J5: LCSC Part # C52995100 -> C160402; MPN WAFA2-RDT1-2021-D -> SM02B-SRSS-TB(LF)(SN)
Changed lines of the file:
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@@
 			)
 		)
-		(property "MPN" "WAFA2-RDT1-2021-D"
+		(property "MPN" "SM02B-SRSS-TB(LF)(SN)"
 			(at 120.65 37.465 0)
 			(effects
@@
 			)
 		)
-		(property "LCSC Part #" "C52995100"
+		(property "LCSC Part #" "C160402"
 			(at 120.65 40.005 0)
 			(effects
